File: Marble_Tiny/PMODs.kicad_sch (KiCad schematic)
At the start: 6 parts, among them J14 Conn_02x06_Counter_Clockwise, J15 Conn_02x06_Counter_Clockwise, J4 Conn_02x06_Counter_Clockwise, J5 Conn_02x06_Counter_Clockwise, J6 Conn_02x06_Counter_Clockwise, J7 Conn_02x06_Counter_Clockwise

Commit message: components placement and PCB routing
Parts:
- removed J14, J15, J4, J5, J6, J7: Conn_02x06_Counter_Clockwise, Connector_PinSocket_2.54mm:PinSocket_2x06_P2.54mm_Horizontal, symbol Connector_Generic:Conn_02x06_Counter_Clockwise
- added J14, J15: Conn_02x06_Odd_Even, Connector_PinSocket_2.54mm:PinSocket_2x06_P2.54mm_Vertical, symbol Connector_Generic:Conn_02x06_Odd_Even
- added J4, J5, J6, J7: Conn_02x06_Odd_Even, Connector_PinSocket_2.54mm:PinSocket_2x06_P2.54mm_Horizontal, symbol Connector_Generic:Conn_02x06_Odd_Even
Connections:
- net +3V3_P: now also J14.11 (Pin_11), J14.12 (Pin_12), J15.11 (Pin_11), J15.12 (Pin_12), J4.11 (Pin_11), J4.12 (Pin_12), J5.11 (Pin_11), J5.12 (Pin_12), J6.11 (Pin_11), J6.12 (Pin_12), J7.11 (Pin_11), J7.12 (Pin_12)
- net GND: now also J14.10 (Pin_10), J14.9 (Pin_9), J15.10 (Pin_10), J15.9 (Pin_9), J4.10 (Pin_10), J4.9 (Pin_9), J5.10 (Pin_10), J5.9 (Pin_9), J6.10 (Pin_10), J6.9 (Pin_9), J7.10 (Pin_10), J7.9 (Pin_9)
- net PMOD1_0: now also J4.1 (Pin_1)
- net PMOD1_1: now also J4.3 (Pin_3)
- net PMOD1_2: now also J4.5 (Pin_5)
- net PMOD1_3: now also J4.7 (Pin_7)
- net PMOD1_4: now also J4.2 (Pin_2)
- net PMOD1_5: now also J4.4 (Pin_4)
- net PMOD1_6: now also J4.6 (Pin_6)
- net PMOD1_7: now also J4.8 (Pin_8)
- net PMOD2_0: now also J5.1 (Pin_1)
- net PMOD2_1: now also J5.3 (Pin_3)
- net PMOD2_2: now also J5.5 (Pin_5)
- net PMOD2_3: now also J5.7 (Pin_7)
- net PMOD2_4: now also J5.2 (Pin_2)
- net PMOD2_5: now also J5.4 (Pin_4)
- net PMOD2_6: now also J5.6 (Pin_6)
- net PMOD2_7: now also J5.8 (Pin_8)
- net PMOD3_0: now also J6.1 (Pin_1)
- net PMOD3_1: now also J6.3 (Pin_3)
- net PMOD3_2: now also J6.5 (Pin_5)
- net PMOD3_3: now also J6.7 (Pin_7)
- net PMOD3_4: now also J6.2 (Pin_2)
- net PMOD3_5: now also J6.4 (Pin_4)
- net PMOD3_6: now also J6.6 (Pin_6)
- net PMOD3_7: now also J6.8 (Pin_8)
- net PMOD4_0: now also J7.1 (Pin_1)
- net PMOD4_1: now also J7.3 (Pin_3)
- net PMOD4_2: now also J7.5 (Pin_5)
- net PMOD4_3: now also J7.7 (Pin_7)
- net PMOD4_4: now also J7.2 (Pin_2)
- net PMOD4_5: now also J7.4 (Pin_4)
- net PMOD4_6: now also J7.6 (Pin_6)
- net PMOD4_7: now also J7.8 (Pin_8)
- net PMOD5_0: now also J14.1 (Pin_1)
- net PMOD5_1: now also J14.3 (Pin_3)
- net PMOD5_2: now also J14.5 (Pin_5)
- net PMOD5_3: now also J14.7 (Pin_7)
- net PMOD5_4: now also J14.2 (Pin_2)
- net PMOD5_5: now also J14.4 (Pin_4)
- net PMOD5_6: now also J14.6 (Pin_6)
- net PMOD5_7: now also J14.8 (Pin_8)
- net PMOD6_0: now also J15.1 (Pin_1)
- net PMOD6_1: now also J15.3 (Pin_3)
- net PMOD6_2: now also J15.5 (Pin_5)
- net PMOD6_3: now also J15.7 (Pin_7)
- net PMOD6_4: now also J15.2 (Pin_2)
- net PMOD6_5: now also J15.4 (Pin_4)
- net PMOD6_6: now also J15.6 (Pin_6)
- net PMOD6_7: now also J15.8 (Pin_8)
