File: Marble_Tiny/PMODs.kicad_sch (KiCad schematic)
At the start: 5 parts, among them J15 Conn_02x06_Top_Bottom, J4 Conn_02x06_Top_Bottom, J5 Conn_02x06_Top_Bottom, J6 Conn_02x06_Top_Bottom, J7 Conn_02x06_Top_Bottom

Commit message: connected more address lines to DDR, new board name
Parts:
- added J15: Conn_02x06_Top_Bottom, Miscellaneous THD:PinSocket_2x06_P2.54mm_Vertical_PMOD, symbol Connector_Generic:Conn_02x06_Top_Bottom
- renumbered J15 to J14
Connections:
- net +3V3_P: now also J15.12 (Pin_12), J15.6 (Pin_6)
- net GND: now also J15.11 (Pin_11), J15.5 (Pin_5)
- net PMOD6_0: now also J15.1 (Pin_1); no longer J14.1 (Pin_1)
- net PMOD6_1: now also J15.2 (Pin_2); no longer J14.2 (Pin_2)
- net PMOD6_2: now also J15.3 (Pin_3); no longer J14.3 (Pin_3)
- net PMOD6_3: now also J15.4 (Pin_4); no longer J14.4 (Pin_4)
- net PMOD6_4: now also J15.7 (Pin_7); no longer J14.7 (Pin_7)
- net PMOD6_5: now also J15.8 (Pin_8); no longer J14.8 (Pin_8)
- net PMOD6_6: now also J15.9 (Pin_9); no longer J14.9 (Pin_9)
- net PMOD6_7: now also J15.10 (Pin_10); no longer J14.10 (Pin_10)
