File: Marble_Tiny/FPGA.kicad_sch (KiCad schematic)
At the start: 41 parts, among them T1 BSS138LT1G, T2 BSS138LT1G, U1 XC7A35T-CSG325

Commit message: components placement and PCB routing
Connections:
- net ARDUINO_D0: now also U1.G14 (IO_L22P_T3_A17_15); no longer U1.B12 (IO_L7P_T1_AD2P_15)
- net ARDUINO_D1: now also U1.H16 (IO_L20P_T3_A20_15); no longer U1.A12 (IO_L7N_T1_AD2N_15)
- net ARDUINO_D10: now also U1.C17 (IO_L18P_T2_A24_15); no longer U1.F18 (IO_L19N_T3_A21_VREF_15)
- net ARDUINO_D11: now also U1.B15 (IO_L9N_T1_DQS_AD3N_15); no longer U1.H16 (IO_L20P_T3_A20_15)
- net ARDUINO_D12: now also U1.B14 (IO_L10P_T1_AD11P_15); no longer U1.G16 (IO_L20N_T3_A19_15)
- net ARDUINO_D13: now also U1.A14 (IO_L8N_T1_AD10N_15); no longer U1.G15 (IO_L21P_T3_DQS_15)
- net ARDUINO_D2: now also U1.A12 (IO_L7N_T1_AD2N_15); no longer U1.A13 (IO_L8P_T1_AD10P_15)
- net ARDUINO_D3: now also U1.B12 (IO_L7P_T1_AD2P_15); no longer U1.A14 (IO_L8N_T1_AD10N_15)
- net ARDUINO_D5: now also U1.G17 (IO_L19P_T3_A22_15); no longer U1.B15 (IO_L9N_T1_DQS_AD3N_15)
- net ARDUINO_D6: now also U1.G16 (IO_L20N_T3_A19_15); no longer U1.B14 (IO_L10P_T1_AD11P_15)
- net ARDUINO_D7: now also U1.A15 (IO_L10N_T1_AD11N_15); no longer U1.C17 (IO_L18P_T2_A24_15)
- net ARDUINO_D9: now also U1.F18 (IO_L19N_T3_A21_VREF_15); no longer U1.G17 (IO_L19P_T3_A22_15)
- net CLK20_VCXO: now also U1.D13 (IO_L11P_T1_SRCC_15); no longer U1.C12 (IO_L6N_T0_VREF_15)
- net DDR3_A0: now also U1.U2 (IO_L15P_T2_DQS_34); no longer U1.R1 (IO_L13N_T2_MRCC_34)
- net DDR3_A1: now also U1.V3 (IO_L16P_T2_34); no longer U1.R3 (IO_L14P_T2_SRCC_34)
- net DDR3_A10: now also U1.U1 (IO_L15N_T2_DQS_34); no longer U1.V4 (IO_L18N_T2_34)
- net DDR3_A11: now also U1.U7 (IO_L23P_T3_34); no longer U1.P6 (IO_L19P_T3_34)
- net DDR3_A12: now also U1.U6 (IO_L20P_T3_34); no longer U1.P5 (IO_L19N_T3_VREF_34)
- net DDR3_A13: now also U1.U5 (IO_L20N_T3_34); no longer U1.U6 (IO_L20P_T3_34)
- net DDR3_A2: now also U1.R7 (IO_L22P_T3_34); no longer U1.T2 (IO_L14N_T2_SRCC_34)
- net DDR3_A3: now also U1.P6 (IO_L19P_T3_34); no longer U1.U2 (IO_L15P_T2_DQS_34)
- net DDR3_A4: now also U1.V2 (IO_L16N_T2_34); no longer U1.U1 (IO_L15N_T2_DQS_34)
- net DDR3_A5: now also U1.V4 (IO_L18N_T2_34); no longer U1.V3 (IO_L16P_T2_34)
- net DDR3_A6: now also U1.V7 (IO_L24N_T3_34); no longer U1.V2 (IO_L16N_T2_34)
- net DDR3_A7: now also U1.T7 (IO_L22N_T3_34); no longer U1.T4 (IO_L17P_T2_34)
- net DDR3_A8: now also U1.V8 (IO_L24P_T3_34); no longer U1.T3 (IO_L17N_T2_34)
- net DDR3_BA0: now also U1.T3 (IO_L17N_T2_34); no longer U1.V6 (IO_L23N_T3_34)
- net DDR3_BA1: now also U1.V6 (IO_L23N_T3_34); no longer U1.V8 (IO_L24P_T3_34)
- net DDR3_BA2: now also U1.R2 (IO_L13P_T2_MRCC_34); no longer U1.V7 (IO_L24N_T3_34)
- net DDR3_CAS: now also U1.T2 (IO_L14N_T2_SRCC_34); no longer U1.P3 (IO_L12N_T1_MRCC_34)
- net DDR3_CE: now also U1.P5 (IO_L19N_T3_VREF_34); no longer U1.U5 (IO_L20N_T3_34)
- net DDR3_CKE0: now also U1.R1 (IO_L13N_T2_MRCC_34); no longer U1.U7 (IO_L23P_T3_34)
- net DDR3_D0: now also U1.K3 (IO_L4P_T0_34); no longer U1.K6 (IO_L1P_T0_34)
- net DDR3_D1: now also U1.L4 (IO_L5P_T0_34); no longer U1.K5 (IO_L1N_T0_34)
- net DDR3_D10: now also U1.N2 (IO_L11N_T1_SRCC_34); no longer U1.M6 (IO_L8P_T1_34)
- net DDR3_D11: now also U1.M4 (IO_L10P_T1_34); no longer U1.N6 (IO_L8N_T1_34)
- net DDR3_D12: now also U1.N6 (IO_L8N_T1_34); no longer U1.M4 (IO_L10P_T1_34)
- net DDR3_D13: now also U1.M2 (IO_L7P_T1_34); no longer U1.N4 (IO_L10N_T1_34)
- net DDR3_D14: now also U1.P4 (IO_L12P_T1_MRCC_34); no longer U1.N3 (IO_L11P_T1_SRCC_34)
- net DDR3_D15: now also U1.N4 (IO_L10N_T1_34); no longer U1.N2 (IO_L11N_T1_SRCC_34)
- net DDR3_D2: now also U1.K5 (IO_L1N_T0_34); no longer U1.J5 (IO_L2P_T0_34)
- net DDR3_D3: now also U1.K6 (IO_L1P_T0_34); no longer U1.J4 (IO_L2N_T0_34)
- net DDR3_D4: now also U1.J4 (IO_L2N_T0_34); no longer U1.K3 (IO_L4P_T0_34)
- net DDR3_D6: now also U1.J5 (IO_L2P_T0_34); no longer U1.L4 (IO_L5P_T0_34)
- net DDR3_D8: now also U1.N3 (IO_L11P_T1_SRCC_34); no longer U1.M2 (IO_L7P_T1_34)
- net DDR3_DM1: now also U1.M6 (IO_L8P_T1_34); no longer U1.P4 (IO_L12P_T1_MRCC_34)
- net DDR3_ODT: now also U1.P3 (IO_L12N_T1_MRCC_34); no longer U1.R7 (IO_L22P_T3_34)
- net DDR3_RAS: now also U1.R3 (IO_L14P_T2_SRCC_34); no longer U1.R2 (IO_L13P_T2_MRCC_34)
- net DDR3_WE: now also U1.T4 (IO_L17P_T2_34); no longer U1.T7 (IO_L22N_T3_34)
- net I2C_SDA_Ardu: now also U1.C12 (IO_L6N_T0_VREF_15); no longer U1.D15 (IO_L13N_T2_MRCC_15)
- net PHY_RSTn: now also U1.A13 (IO_L8P_T1_AD10P_15); no longer U1.A15 (IO_L10N_T1_AD11N_15)
- net PMOD1_0: now also U1.U16 (IO_L17N_T2_A13_D29_14); no longer U1.L14 (IO_0_14)
- net PMOD1_1: now also U1.R18 (IO_L15P_T2_DQS_RDWR_B_14); no longer U1.F15 (IO_L21N_T3_DQS_A18_15)
- net PMOD1_2: now also U1.N17 (IO_L9N_T1_DQS_D13_14); no longer U1.G14 (IO_L22P_T3_A17_15)
- net PMOD1_3: now also U1.M16 (IO_L7P_T1_D09_14); no longer U1.J15 (IO_L2P_T0_D02_14)
- net PMOD1_4: now also U1.V17 (IO_L18N_T2_A11_D27_14); no longer U1.J16 (IO_L2N_T0_D03_14)
- net PMOD1_5: now also U1.P18 (IO_L10N_T1_D15_14); no longer U1.K18 (IO_L3N_T0_DQS_EMCCLK_14)
- net PMOD1_6: now also U1.N18 (IO_L10P_T1_D14_14); no longer U1.K17 (IO_L4P_T0_D04_14)
- net PMOD1_7: now also U1.M17 (IO_L7N_T1_D10_14); no longer U1.L18 (IO_L4N_T0_D05_14)
- net PMOD2_0: now also U1.V14 (IO_L20N_T3_A07_D23_14); no longer U1.J14 (IO_L5P_T0_D06_14)
- net PMOD2_1: now also U1.U15 (IO_L17P_T2_A14_D30_14); no longer U1.K15 (IO_L5N_T0_D07_14)
- net PMOD2_2: now also U1.U17 (IO_L16N_T2_A15_D31_14); no longer U1.M15 (IO_L6N_T0_D08_VREF_14)
- net PMOD2_3: now also U1.T18 (IO_L15N_T2_DQS_DOUT_CSO_B_14); no longer U1.M16 (IO_L7P_T1_D09_14)
- net PMOD2_4: now also U1.U14 (IO_L20P_T3_A08_D24_14); no longer U1.M17 (IO_L7N_T1_D10_14)
- net PMOD2_5: now also U1.V16 (IO_L18P_T2_A12_D28_14); no longer U1.M14 (IO_L8P_T1_D11_14)
- net PMOD2_6: now also U1.T17 (IO_L16P_T2_CSI_B_14); no longer U1.N14 (IO_L8N_T1_D12_14)
- net PMOD2_7: now also U1.R17 (IO_L14N_T2_SRCC_14); no longer U1.N16 (IO_L9P_T1_DQS_14)
- net PMOD3_0: now also U1.L18 (IO_L4N_T0_D05_14); no longer U1.N17 (IO_L9N_T1_DQS_D13_14)
- net PMOD3_1: now also U1.K17 (IO_L4P_T0_D04_14); no longer U1.N18 (IO_L10P_T1_D14_14)
- net PMOD3_2: now also U1.P16 (IO_L11N_T1_SRCC_14); no longer U1.P18 (IO_L10N_T1_D15_14)
- net PMOD3_3: now also U1.N14 (IO_L8N_T1_D12_14); no longer U1.P15 (IO_L11P_T1_SRCC_14)
- net PMOD3_4: now also U1.K18 (IO_L3N_T0_DQS_EMCCLK_14); no longer U1.P16 (IO_L11N_T1_SRCC_14)
- net PMOD3_5: now also U1.P15 (IO_L11P_T1_SRCC_14); no longer U1.P14 (IO_L12P_T1_MRCC_14)
- net PMOD3_6: now also U1.N16 (IO_L9P_T1_DQS_14); no longer U1.R15 (IO_L12N_T1_MRCC_14)
- net PMOD3_7: now also U1.M15 (IO_L6N_T0_D08_VREF_14); no longer U1.T14 (IO_L13P_T2_MRCC_14)
- net PMOD4_0: now also U1.K15 (IO_L5N_T0_D07_14); no longer U1.T15 (IO_L13N_T2_MRCC_14)
- net PMOD4_1: now also U1.J16 (IO_L2N_T0_D03_14); no longer U1.R16 (IO_L14P_T2_SRCC_14)
- net PMOD4_2: now also U1.J14 (IO_L5P_T0_D06_14); no longer U1.R17 (IO_L14N_T2_SRCC_14)
- net PMOD4_3: now also U1.F15 (IO_L21N_T3_DQS_A18_15); no longer U1.R18 (IO_L15P_T2_DQS_RDWR_B_14)
- net PMOD4_4: now also U1.M14 (IO_L8P_T1_D11_14); no longer U1.T18 (IO_L15N_T2_DQS_DOUT_CSO_B_14)
- net PMOD4_5: now also U1.J15 (IO_L2P_T0_D02_14); no longer U1.T17 (IO_L16P_T2_CSI_B_14)
- net PMOD4_6: now also U1.L14 (IO_0_14); no longer U1.U17 (IO_L16N_T2_A15_D31_14)
- net PMOD4_7: now also U1.G15 (IO_L21P_T3_DQS_15); no longer U1.U15 (IO_L17P_T2_A14_D30_14)
- net PMOD5_0: now also U1.V11 (IO_L23N_T3_A02_D18_14); no longer U1.U16 (IO_L17N_T2_A13_D29_14)
- net PMOD5_1: now also U1.V9 (IO_L24N_T3_A00_D16_14); no longer U1.V16 (IO_L18P_T2_A12_D28_14)
- net PMOD5_2: now also U1.U9 (IO_L24P_T3_A01_D17_14); no longer U1.V17 (IO_L18N_T2_A11_D27_14)
- net PMOD5_3: now also U1.U10 (IO_25_14); no longer U1.R13 (IO_L19P_T3_A10_D26_14)
- net PMOD5_4: now also U1.U11 (IO_L23P_T3_A03_D19_14); no longer U1.T13 (IO_L19N_T3_A09_D25_VREF_14)
- net PMOD5_5: now also U1.V13 (IO_L21N_T3_DQS_A06_D22_14); no longer U1.U14 (IO_L20P_T3_A08_D24_14)
- net PMOD5_6: now also U1.U12 (IO_L22N_T3_A04_D20_14); no longer U1.V14 (IO_L20N_T3_A07_D23_14)
- net PMOD6_0: now also U1.T14 (IO_L13P_T2_MRCC_14); no longer U1.V13 (IO_L21N_T3_DQS_A06_D22_14)
- net PMOD6_1: now also U1.R13 (IO_L19P_T3_A10_D26_14); no longer U1.T12 (IO_L22P_T3_A05_D21_14)
- net PMOD6_2: now also U1.T12 (IO_L22P_T3_A05_D21_14); no longer U1.U12 (IO_L22N_T3_A04_D20_14)
- net PMOD6_3: now also U1.T13 (IO_L19N_T3_A09_D25_VREF_14); no longer U1.U11 (IO_L23P_T3_A03_D19_14)
- net PMOD6_4: now also U1.R15 (IO_L12N_T1_MRCC_14); no longer U1.V11 (IO_L23N_T3_A02_D18_14)
- net PMOD6_5: now also U1.R16 (IO_L14P_T2_SRCC_14); no longer U1.U9 (IO_L24P_T3_A01_D17_14)
- net PMOD6_6: now also U1.P14 (IO_L12P_T1_MRCC_14); no longer U1.V9 (IO_L24N_T3_A00_D16_14)
- net PMOD6_7: now also U1.T15 (IO_L13N_T2_MRCC_14); no longer U1.U10 (IO_25_14)
- net RGMII_RXD0: now also U1.B16 (IO_L15P_T2_DQS_15); no longer U1.E16 (IO_L14P_T2_SRCC_15)
- net RGMII_RXD1: now also U1.C16 (IO_L16P_T2_A28_15); no longer U1.D16 (IO_L14N_T2_SRCC_15)
- net RGMII_RXD2: now also U1.D14 (IO_L12N_T1_MRCC_15); no longer U1.B16 (IO_L15P_T2_DQS_15)
- net RGMII_RXD3: now also U1.C13 (IO_L11N_T1_SRCC_15); no longer U1.A17 (IO_L15N_T2_DQS_ADV_B_15)
- net RGMII_RX_DV: now also U1.D16 (IO_L14N_T2_SRCC_15); no longer U1.D14 (IO_L12N_T1_MRCC_15)
- net RGMII_TXD0: now also U1.B17 (IO_L16N_T2_A27_15); no longer U1.C16 (IO_L16P_T2_A28_15)
- net RGMII_TXD1: now also U1.E16 (IO_L14P_T2_SRCC_15); no longer U1.B17 (IO_L16N_T2_A27_15)
- net RGMII_TX_CLK: now also U1.D15 (IO_L13N_T2_MRCC_15); no longer U1.D13 (IO_L11P_T1_SRCC_15)
- net RGMII_TX_EN: now also U1.A17 (IO_L15N_T2_DQS_ADV_B_15); no longer U1.C13 (IO_L11N_T1_SRCC_15)

Commit message: PCB done
Parts:
- added TP2, TP3: TestPoint, TestPoint:TestPoint_THTPad_D1.5mm_Drill0.7mm, symbol Connector_Generic:TestPoint
- renumbered B6 to U28
Connections:
- net I2C_SCL: now also TP2.1
- net I2C_SDA: now also TP3.1
Changed lines of the file:
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@@
 	(wire
 		(pts
+			(xy 191.77 229.87) (xy 191.77 232.41)
+		)
+		(stroke
+			(width 0)
+			(type default)
+		)
+	)
+	(wire
+		(pts
 			(xy 350.52 107.95) (xy 369.57 107.95)
 		)
@@
 	(wire
 		(pts
+			(xy 190.5 229.87) (xy 191.77 229.87)
+		)
+		(stroke
+			(width 0)
+			(type default)
+		)
+	)
+	(wire
+		(pts
 			(xy 100.33 66.04) (xy 102.87 66.04)
 		)
@@
 	(wire
 		(pts
-			(xy 193.04 234.95) (xy 212.09 234.95)
-		)
-		(stroke
-			(width 0)
-			(type default)
-		)
-	)
-	(wire
-		(pts
 			(xy 71.12 182.88) (xy 90.17 182.88)
 		)
@@
 	(wire
 		(pts
+			(xy 190.5 234.95) (xy 212.09 234.95)
+		)
+		(stroke
+			(width 0)
+			(type default)
+		)
+	)
+	(wire
+		(pts
 			(xy 350.52 166.37) (xy 369.57 166.37)
 		)
@@
 	(wire
 		(pts
+			(xy 191.77 232.41) (xy 203.2 232.41)
+		)
+		(stroke
+			(width 0)
+			(type default)
+		)
+	)
+	(wire
+		(pts
 			(xy 73.66 59.69) (xy 81.28 59.69)
 		)
@@
 	(wire
 		(pts
-			(xy 193.04 232.41) (xy 203.2 232.41)
-		)
-		(stroke
-			(width 0)
-			(type default)
-		)
-	)
-	(wire
-		(pts
 			(xy 191.77 137.16) (xy 214.63 137.16)
 		)
@@
 		(on_board yes)
 		(dnp no)
-		(property "Reference" "B6"
+		(property "Reference" "U28"
 			(at 139.7 229.87 0)
 			(effects
@@
 			(project "Marble_Tiny"
 				(path "/c2a4f786-b14c-434a-acf7-b20fb2221b0b/26bc6f09-ebb0-4c32-8a32-ec70c3f97c4f"
-					(reference "B6")
+					(reference "U28")
+					(unit 1)
+				)
+			)
+		)
+	)
+	(symbol
+		(lib_id "Connector_Generic:TestPoint")
+		(at 190.5 234.95 90)
+		(mirror x)
+		(unit 1)
+		(exclude_from_sim no)
+		(in_bom yes)
+		(on_board yes)
+		(dnp no)
+		(property "Reference" "TP2"
+			(at 185.674 235.204 90)
+			(effects
+				(font
+					(size 1.27 1.27)
+				)
+				(justify left)
+			)
+		)
+		(property "Value" "TestPoint"
+			(at 190.246 237.236 90)
+			(effects
+				(font
+					(size 1.27 1.27)
+				)
+				(justify left)
+			)
+		)
+		(property "Footprint" "TestPoint:TestPoint_THTPad_D1.5mm_Drill0.7mm"
+			(at 190.5 240.03 0)
+			(effects
+				(font
+					(size 1.27 1.27)
+				)
+				(hide yes)
+			)
+		)
+		(property "Datasheet" ""
+			(at 190.5 240.03 0)
+			(effects
+				(font
+					(size 1.27 1.27)
+				)
+				(hide yes)
+			)
+		)
+		(property "Description" ""
+			(at 190.5 234.95 0)
+			(effects
+				(font
+					(size 1.27 1.27)
+				)
+				(hide yes)
+			)
+		)
+		(pin "1"
+		)
+		(instances
+			(project "Marble_Tiny"
+				(path "/c2a4f786-b14c-434a-acf7-b20fb2221b0b/26bc6f09-ebb0-4c32-8a32-ec70c3f97c4f"
+					(reference "TP2")
 					(unit 1)
 				)
@@
 					(unit 1)
 				)
+			)
+		)
+	)
+	(symbol
+		(lib_id "Connector_Generic:TestPoint")
+		(at 190.5 229.87 90)
+		(mirror x)
+		(unit 1)
+		(exclude_from_sim no)
+		(in_bom yes)
+		(on_board yes)
+		(dnp no)
+		(property "Reference" "TP3"
+			(at 185.674 230.124 90)
+			(effects
+				(font
+					(size 1.27 1.27)
+				)
+				(justify left)
+			)
+		)
+		(property "Value" "TestPoint"
+			(at 190.246 232.156 90)
+			(effects
+				(font
+					(size 1.27 1.27)
+				)
+				(justify left)
+			)
+		)
+		(property "Footprint" "TestPoint:TestPoint_THTPad_D1.5mm_Drill0.7mm"
+			(at 190.5 234.95 0)
+			(effects
+				(font
+					(size 1.27 1.27)
+				)
+				(hide yes)
+			)
+		)
+		(property "Datasheet" ""
+			(at 190.5 234.95 0)
+			(effects
+				(font
+					(size 1.27 1.27)
+				)
+				(hide yes)
+			)
+		)
+		(property "Description" ""
+			(at 190.5 229.87 0)
+			(effects
+				(font
+					(size 1.27 1.27)
+				)
+				(hide yes)
+			)
+		)
+		(pin "1"
+		)
+		(instances
+			(project "Marble_Tiny"
+				(path "/c2a4f786-b14c-434a-acf7-b20fb2221b0b/26bc6f09-ebb0-4c32-8a32-ec70c3f97c4f"
+					(reference "TP3")
+					(unit 1)
+				)
