File: Marble_Tiny/FPGA_MISC.kicad_sch (KiCad schematic)
At the start: 17 parts, among them IC3 S25FL128SAGMFI001, U1 XC7A35T-CSG325, U9 REF3012

Commit message: components placement and PCB routing
Parts:
- added LD5: LED_KINGBRIGHT_KPH-1608CGCK, ICs And Semiconductors SMD:LED_KINGBRIGHT_KPH-1608CGCK, symbol LEDs & Displays:LED_KINGBRIGHT_KPH-1608CGCK
- added R161: R0402_10K_1%_0.0625W_100PPM, Resistors SMD:RESC1005X40N, symbol Resistors SMD:R0402_10K_1%_0.0625W_100PPM
- added T3: BSS138LT1G, ICs And Semiconductors SMD:SOT95P240X110-3N, symbol Transistors:BSS138LT1G
Connections:
- net +3V3: now also R161.2
- net GND: now also T3.2 (S)
- net at U1.F12 (DONE_0): now also T3.1 (G)
- new net: LD5.2 (A), R161.1
- new net: LD5.1 (C), T3.3 (D)
Other:
- note added: "FPGA DONE"

Commit message: PCB done
Parts:
- removed C154: CC0201_10NF_10V_10%_X5R, Capacitors SMD:CAPC0603X33N, symbol Capacitors SMD:CC0201_10NF_10V_10%_X5R
- added C154: CC0201_100NF_6.3V_10%_X5R, Capacitors SMD:CAPC0603X33N, symbol Capacitors_SMD:CC0201_100NF_6.3V_10%_X5R
- renumbered IC3 to U27
Connections:
- net VREF: now also C154.2
- net XADCGND: now also C154.1
