File: Marble_Tiny/FPGA_MISC.kicad_sch (KiCad schematic)
At the start: 21 parts, among them SW1 SW_DIP_x01, T3 BSS138LT1G, U1 XC7A35T-CSG325, U27 S25FL128SAGMFI001, U9 REF3012

Commit message: ready for the final review
Parts:
- renumbered T3 to Q3
Changed lines of the file:
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@@
 		(dnp no)
 		(fields_autoplaced yes)
-		(property "Reference" "T3"
+		(property "Reference" "Q3"
 			(at 256.54 123.1899 0)
 			(effects
@@
 			(project ""
 				(path "/c2a4f786-b14c-434a-acf7-b20fb2221b0b/74b17685-a06b-496e-ad9c-4554e740129f"
-					(reference "T3")
+					(reference "Q3")
 					(unit 1)
 				)
