File: Marble_Tiny/SFP.kicad_sch (KiCad schematic)
At the start: 73 parts, among them IC4 PCA9546ARGV, J1 TYCO_1888247-1, J11 TYCO_1888247-1, J12 TYCO_1888247-1, J13 TYCO_1888247-1, J8 2180739-1, J9 2180739-1, U17 TCA9535RTWR, U19 TCA9535RTWR

Commit message: PCB done
Parts:
- renumbered IC4 to U26
Changed lines of the file:
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@@
 		(on_board yes)
 		(dnp no)
-		(property "Reference" "IC4"
+		(property "Reference" "U26"
 			(at 336.55 172.72 0)
 			(effects
@@
 			(project ""
 				(path "/c2a4f786-b14c-434a-acf7-b20fb2221b0b/f19bf9c4-473e-4b3f-a56f-356b0388d57c"
-					(reference "IC4")
+					(reference "U26")
 					(unit 1)
 				)
