File: Marble_Tiny/USB.kicad_sch (KiCad schematic)
At the start: 40 parts, among them IC1 FT2232HQ, IC2 93C46B-I_SN, J2 USB_C_Receptacle_USB2.0_16P, Q2 XTAL_12MHZ_TXC_7A-12.000MAAJ-T, U8 TLV62565DBV

Commit message: components placement and PCB routing
Connections:
- net USB_N: now reaches D1.3 (I/O2), IC1.7 (DM), J2.A7 (D-), J2.B7 (D-)
- net USB_P: now reaches D1.2 (I/O1), IC1.8 (DP), J2.A6 (D+), J2.B6 (D+)
- net TCK renamed JTAG_TCK
- net TDI renamed JTAG_TDI
- net TDO renamed JTAG_TDO
- net TMS renamed JTAG_TMS
Changed lines of the file:
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@@
+		)
+	)
+	(label "USB_N"
+		(at 69.85 45.72 0)
+		(effects
+			(font
+				(size 1.27 1.27)
+			)
+			(justify left bottom)
 		)
 	)
@@
 		)
 	)
+	(label "USB_P"
+		(at 69.85 50.8 0)
+		(effects
+			(font
+				(size 1.27 1.27)
+			)
+			(justify left bottom)
+		)
+	)
 	(label "USB_TDO_DI"
 		(at 223.52 34.29 0)
@@
 			)
 			(justify left bottom)
+		)
+	)
+	(global_label "JTAG_TDO"
+		(shape input)
+		(at 243.84 34.29 0)
+		(fields_autoplaced yes)
+		(effects
+			(font
+				(size 1.27 1.27)
+			)
+			(justify left)
+		)
+		(property "Intersheetrefs" "${INTERSHEET_REFS}"
+			(at 255.6547 34.29 0)
+			(effects
+				(font
+					(size 1.27 1.27)
+				)
+				(justify left)
+				(hide yes)
+			)
+		)
+	)
+	(global_label "JTAG_TMS"
+		(shape output)
+		(at 243.84 36.83 0)
+		(fields_autoplaced yes)
+		(effects
+			(font
+				(size 1.27 1.27)
+			)
+			(justify left)
+		)
+		(property "Intersheetrefs" "${INTERSHEET_REFS}"
+			(at 255.7151 36.83 0)
+			(effects
+				(font
+					(size 1.27 1.27)
+				)
+				(justify left)
+				(hide yes)
+			)
 		)
 	)
@@
 		)
 	)
-	(global_label "TCK"
+	(global_label "JTAG_TDI"
 		(shape output)
-		(at 243.84 29.21 0)
+		(at 243.84 31.75 0)
 		(fields_autoplaced yes)
 		(effects
@@
 		)
 		(property "Intersheetrefs" "${INTERSHEET_REFS}"
-			(at 250.3328 29.21 0)
-			(effects
-				(font
-					(size 1.27 1.27)
-				)
-				(justify left)
-				(hide yes)
-			)
-		)
-	)
-	(global_label "TDO"
-		(shape input)
-		(at 243.84 34.29 0)
-		(fields_autoplaced yes)
-		(effects
-			(font
-				(size 1.27 1.27)
-			)
-			(justify left)
-		)
-		(property "Intersheetrefs" "${INTERSHEET_REFS}"
-			(at 250.3933 34.29 0)
+			(at 254.929 31.75 0)
 			(effects
 				(font
@@
 		)
 	)
-	(global_label "TDI"
+	(global_label "JTAG_TCK"
 		(shape output)
-		(at 243.84 31.75 0)
+		(at 243.84 29.21 0)
 		(fields_autoplaced yes)
 		(effects
@@
 		)
 		(property "Intersheetrefs" "${INTERSHEET_REFS}"
-			(at 249.6676 31.75 0)
+			(at 255.5942 29.21 0)
 			(effects
 				(font
-					(size 1.27 1.27)
-				)
-				(justify left)
-				(hide yes)
-			)
-		)
-	)
-	(global_label "TMS"
-		(shape output)
-		(at 243.84 36.83 0)
-		(fields_autoplaced yes)
-		(effects
-			(font
-				(size 1.27 1.27)
-			)
-			(justify left)
-		)
-		(property "Intersheetrefs" "${INTERSHEET_REFS}"
-			(at 250.4537 36.83 0)
-			(effects
-				(font

Commit message: PCB done
Parts:
- renumbered IC1 to U21, IC2 to U22
Changed lines of the file:
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@@
 			)
 		)
-		(property "Datasheet" " "
+		(property "Datasheet" ""
 			(at 121.92 114.3 0)
 			(effects
@@
 		(on_board yes)
 		(dnp no)
-		(property "Reference" "IC2"
+		(property "Reference" "U22"
 			(at 134.366 71.12 0)
 			(effects
@@
 			(project ""
 				(path "/c2a4f786-b14c-434a-acf7-b20fb2221b0b/62565c75-62b0-4544-832f-1275174835af"
-					(reference "IC2")
+					(reference "U22")
 					(unit 1)
 				)
@@
 		(on_board yes)
 		(dnp no)
-		(property "Reference" "IC1"
+		(property "Reference" "U21"
 			(at 201.93 24.13 0)
 			(effects
@@
 			(project "Marble_Tiny"
 				(path "/c2a4f786-b14c-434a-acf7-b20fb2221b0b/62565c75-62b0-4544-832f-1275174835af"
-					(reference "IC1")
+					(reference "U21")
 					(unit 1)
 				)
