File: Marble_Tiny/untitled.kicad_sch (KiCad schematic)
At the start: 67 parts, among them Q3 XTAL_25MHZ_TXC_8Y-25.000MAAJ-T, U12 LP5951MF-3.0/NOPB, U13 LM336M-2.5, U14 DAC8550IDGK, U15 DAC8550IDGK, U16 CDCM61004RHB, U3 Si5351A-B-GT, Y1 OSC_25MHZ_RAKON_IVT3205CR, Y2 VM53S3-25.000-2.5/-30+75, Y3 OSC_20MHZ_IQD_LFVCXO026156

Commit message: components placement and PCB routing
Parts:
- added R159: R0402_40R2_1%_0.0625W_100PPM, Resistors SMD:RESC1005X40N, symbol Resistors SMD:R0402_40R2_1%_0.0625W_100PPM
Connections:
- net WR_CLK0_N: no longer C213.2, R118.1, U16.5 (OUTN0)
- net WR_CLK0_P: no longer C205.2, R119.1, U16.6 (OUTP0)
- net at U16.23 (OSCOUT): now also R159.1
- new net CLK_25MHZ: R159.2
- new net WRCLK0_N: C213.2, R118.1, U16.5 (OUTN0)
- new net WRCLK0_P: C205.2, R119.1, U16.6 (OUTP0)
- no-connect marks 11 -> 10

Commit message: PCB done
Parts:
- removed C188: CC0402_10NF_16V_10%_X7R, CAPC1005X55N, symbol Capacitors_SMD:CC0402_10NF_16V_10%_X7R
- removed C202: CC0402_100NF_25V_10%_X5R, CAPC1005X55N, symbol Capacitors_SMD:CC0402_100NF_25V_10%_X5R
- added C188: CC0201_100NF_6.3V_10%_X5R, Capacitors SMD:CAPC0603X33N, symbol Capacitors_SMD:CC0201_100NF_6.3V_10%_X5R
- added C202, C248: CC0402_100NF_50V_10%_X7R, Capacitors SMD:CAPC1005X55N, symbol Capacitors SMD:CC0402_100NF_50V_10%_X7R
- added R162: R0402_30K_1%_0.0625W_100PPM, Resistors SMD:RESC1005X40N, symbol Resistors SMD:R0402_30K_1%_0.0625W_100PPM
- added R163: R0402_10K_1%_0.0625W_100PPM, Resistors SMD:RESC1005X40N, symbol Resistors SMD:R0402_10K_1%_0.0625W_100PPM
- C183, C185, C186, C189, C190, C191, C194, C196, C197, C198, C206, C208, C209, C210, C211, C212, C215: footprint CAPC0603X33N -> Capacitors SMD:CAPC0603X33N
Connections:
- net +3V3: now also C198.1, U3.1 (VDD)
- net +3V3_CLEAN: no longer C198.1, U3.1 (VDD)
- net CLK_25MHZ: now also R162.1
- net GND: now also C188.2, C202.2, R163.1
- net at C184.1, C186.1, U12.5 (VOUT)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: now also C188.1
- net at Q3.1 (X), U3.2 (XA): now also C248.1
- net at U16.12 (~{RSTN}): now also C202.1
- new net: C248.2, R162.2, R163.2
