File: Marble_Tiny/Arduino.kicad_sch (KiCad schematic)
At the start: 17 parts

Commit message: ready for the final review
Connections:
- net +3V3_P: now also A1.2 (IOREF)
- no-connect marks 4 -> 3
Changed lines of the file:
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@@
 	)
 	(no_connect
-		(at 151.13 74.93)
-	)
-	(no_connect
 		(at 151.13 80.01)
 	)
@@
 	(wire
 		(pts
+			(xy 151.13 74.93) (xy 157.48 74.93)
+		)
+		(stroke
+			(width 0)
+			(type default)
+		)
+	)
+	(wire
+		(pts
 			(xy 154.94 97.79) (xy 157.48 97.79)
 		)
@@
 		(on_board yes)
 		(dnp no)
-		(fields_autoplaced yes)
 		(property "Reference" "#PWR0295"
 			(at 135.89 63.5 0)
@@
 		)
 		(property "Value" "+12V"
-			(at 135.89 54.61 0)
+			(at 134.366 56.388 0)
 			(effects
 				(font
@@
 	)
 	(symbol
+		(lib_id "power:+1V0")
+		(at 157.48 74.93 0)
+		(unit 1)
+		(exclude_from_sim no)
+		(in_bom yes)
+		(on_board yes)
+		(dnp no)
+		(property "Reference" "#PWR0352"
+			(at 157.48 78.74 0)
+			(effects
+				(font
+					(size 1.27 1.27)
+				)
+				(hide yes)
+			)
+		)
+		(property "Value" "+3V3_P"
+			(at 157.734 71.374 0)
+			(effects
+				(font
+					(size 1.27 1.27)
+				)
+			)
+		)
+		(property "Footprint" ""
+			(at 157.48 74.93 0)
+			(effects
+				(font
+					(size 1.27 1.27)
+				)
+				(hide yes)
+			)
+		)
+		(property "Datasheet" ""
+			(at 157.48 74.93 0)
+			(effects
+				(font
+					(size 1.27 1.27)
+				)
+				(hide yes)
+			)
+		)
+		(property "Description" "Power symbol creates a global label with name \"+1V0\""
+			(at 157.48 74.93 0)
+			(effects
+				(font
+					(size 1.27 1.27)
+				)
+				(hide yes)
+			)
+		)
+		(pin "1"
+		)
+		(instances
+			(project "Marble_Tiny"
+				(path "/c2a4f786-b14c-434a-acf7-b20fb2221b0b/37c76a7d-e360-409e-9f8e-819f870af943"
+					(reference "#PWR0352")
+					(unit 1)
+				)
+			)
+		)
+	)
+	(symbol
 		(lib_id "power:GND")
 		(at 228.6 118.11 0)
@@
 		)
 		(property "Value" "+3V3_P"
-			(at 141.224 56.134 0)
+			(at 142.494 56.134 0)
 			(effects
 				(font
