File: Marble_Tiny/Power.kicad_sch (KiCad schematic)
At the start: 84 parts, among them J10 Barrel_Jack_Switch, Q4 DMP3013SFV, SW3 SW_DIP_x01, U10 TPSM863257RDXR, U11 TPSM863257RDXR, U18 TLV77325PDBVR, U20 RT9045AGSP / AP2303, U23 NCV59801CML120TCG, U24 SN74LVC1G07DBV, U25 SN74LVC1G07DBV, U4 TPSM863257RDXR, U5 TPSM863257RDXR, U6 TPSM863257RDXR

Commit message: minor changes
Parts:
- removed D4: SS38, Diode_SMD:D_SMA, symbol Diode:SS38
- removed D6: DZ2S030X0L, Diode_SMD:D_SOD-523, symbol Diode:DZ2S030X0L
- removed LD1: LED_KINGBRIGHT_KPH-1608CGCK, ICs And Semiconductors SMD:LED_KINGBRIGHT_KPH-1608CGCK, symbol LEDs & Displays:LED_KINGBRIGHT_KPH-1608CGCK
- removed R111, R112: R0402_40R2_1%_0.0625W_100PPM, Resistors SMD:RESC1005X40N, symbol Resistors SMD:R0402_40R2_1%_0.0625W_100PPM
- removed R148: R0402_4K7_1%_0.0625W_100PPM, Resistors SMD:RESC1005X40N, symbol Resistors SMD:R0402_4K7_1%_0.0625W_100PPM
- removed R196: R0402_360K_1%_0.0625W_100PPM, Resistors SMD:RESC1005X40N, symbol Resistors SMD old:R0402_360K_1%_0.0625W_100PPM
- removed R91: R0402_220K_1%_0.0625W_100PPM, Resistors SMD:RESC1005X40N, symbol Resistors SMD old:R0402_220K_1%_0.0625W_100PPM
- removed SW3: SW_DIP_x01, Switches:SW_OMRON_A6SN-1101, symbol Switch:SW_DIP_x01
- added LD1: LED_OSRAM_LS_Q976-NR-1, ICs And Semiconductors SMD:LED_OSRAM_LS Q976, symbol LEDs & Displays:LED_OSRAM_LS_Q976-NR-1
- added R147: R0402_30K_1%_0.0625W_100PPM, Resistors SMD:RESC1005X40N, symbol Resistors SMD:R0402_30K_1%_0.0625W_100PPM
- added R148: R0402_10K_1%_0.0625W_100PPM, Resistors SMD:RESC1005X40N, symbol Resistors SMD:R0402_10K_1%_0.0625W_100PPM
- added R91: R0805_135K_0.1%_0.1W_25PPM_KOA_RN73R2ATTD1353B25, Resistors SMD:RESC2012X60N, symbol Resistors SMD:R0805_135K_0.1%_0.1W_25PPM_KOA_RN73R2ATTD1353B25
Connections:
- net +12V: now also R147.1
- net +3V3: now also R148.2
- net +3V3_P: now also R91.1
- net at C179.2, R92.1, U6.7 (FB): now also R91.2
- net at D3.1 (K), TP6.1, U11.5 (PG)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: now also LD1.1 (C)
- net at LD2.2 (A), U25.4 (OUT): now also R148.1
- new net: LD1.2 (A), R147.2
Other:
- note added: "POWER SUPPLY FAIL"
- note removed: "PMOD VCC SW3 3.3V ON -> 5.0V OFF"
