File: Obsidian/Arduino.kicad_sch (KiCad schematic)
At the start: 17 parts

Commit message: revison v1.1.0 ready to review
Connections:
- net +3V3_P: now also A1.5 (+5V); no longer A1.4 (3V3)
- new net +3V3: A1.4 (3V3)
- no-connect marks 3 -> 2
Changed lines of the file:
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@@
 		(at 151.13 80.01)
 	)
-	(no_connect
-		(at 143.51 59.69)
-	)
 	(wire
 		(pts
@@
 	(wire
 		(pts
+			(xy 143.51 59.69) (xy 148.59 59.69)
+		)
+		(stroke
+			(width 0)
+			(type default)
+		)
+	)
+	(wire
+		(pts
 			(xy 119.38 100.33) (xy 125.73 100.33)
 		)
@@
 		(on_board yes)
 		(dnp no)
-		(property "Reference" "#PWR0294"
+		(property "Reference" "#PWR0209"
 			(at 140.97 63.5 0)
 			(effects
@@
 			)
 		)
-		(property "Value" "+3V3_P"
-			(at 142.494 56.134 0)
+		(property "Value" "+3V3"
+			(at 140.97 56.134 0)
 			(effects
 				(font
@@
 			(effects
 				(font
+					(size 1.27 1.27)
+				)
+				(hide yes)
+			)
+		)
+		(pin "1"
+		)
+		(instances
+			(project "Obsidian"
+				(path "/c2a4f786-b14c-434a-acf7-b20fb2221b0b/37c76a7d-e360-409e-9f8e-819f870af943"
+					(reference "#PWR0209")
+					(unit 1)
+				)
+			)
+		)
+	)
+	(symbol
+		(lib_id "power:+1V0")
+		(at 148.59 59.69 0)
+		(unit 1)
+		(exclude_from_sim no)
+		(in_bom yes)
+		(on_board yes)
+		(dnp no)
+		(property "Reference" "#PWR0294"
+			(at 148.59 63.5 0)
+			(effects
+				(font
+					(size 1.27 1.27)
+				)
+				(hide yes)
+			)
+		)
+		(property "Value" "+3V3_P"
+			(at 150.114 56.134 0)
+			(effects
+				(font
+					(size 1.27 1.27)
+				)
+			)
+		)
+		(property "Footprint" ""
+			(at 148.59 59.69 0)
+			(effects
+				(font
+					(size 1.27 1.27)
+				)
+				(hide yes)
+			)
+		)
+		(property "Datasheet" ""
+			(at 148.59 59.69 0)
+			(effects
+				(font
+					(size 1.27 1.27)
+				)
+				(hide yes)
+			)
+		)
+		(property "Description" "Power symbol creates a global label with name \"+1V0\""
+			(at 148.59 59.69 0)
+			(effects
+				(font
