File: Obsidian/untitled.kicad_sch (KiCad schematic)
At the start: 72 parts, among them U12 LP5951MF-3.0/NOPB, U13 LM336M-2.5, U14 DAC8550IDGK, U15 DAC8550IDGK, U16 CDCM61004RHB, U3 Si5351A-B-GT, Y1 OSC_25MHZ_RAKON_IVT3205CR, Y2 VM53S3-25.000-2.5/-30+75, Y3 OSC_20MHZ_IQD_LFVCXO026156, Y6 XTAL_25MHZ_TXC_8Y-25.000MAAJ-T

Commit message: adding 3D files, 3D model of twist, and correct DRC
Parts:
- C182, C184, C188, C193, C207: footprint Footprint:CAPC1005X55N -> Capacitor_SMD:C_0402_1005Metric; Database Table Name (none) -> Capacitors; Footprint Library (none) -> Capacitors SMD; HelpURL (none) -> \\cern.ch\dfs\Applications\Altium\Datasheets\CC0402_MURATA_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
- C183, C185, C186, C189, C190, C191, C194, C196, C197, C198, C206, C208, C209, C210, C211, C212, C215: Database Table Name (none) -> Capacitors; Footprint Library (none) -> Capacitors SMD; HelpURL (none) -> \\cern.ch\dfs\Applications\Altium\Datasheets\CC0201_X5R_AVX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
- C202, C204, C205, C213, C214, C248: footprint Footprint:CAPC1005X55N -> Capacitor_SMD:C_0402_1005Metric
- R102, R103, R99: Database Table Name (none) -> Resistors; Footprint Library (none) -> Resistors SMD; HelpURL (none) -> \\cern.ch\dfs\Applications\Altium\Datasheets\R0402_Phycomp_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
- U13: Author (none) -> CERN DEM BC; Bonding (none) -> No; Case (none) -> SOIC8; Comment (none) -> 93C46B-I/SN; Component Kind (none) -> Standard; Component Type (none) -> Standard; ComponentHeight (none) -> 1.75mm; ComponentLink1Description (none) -> (none); ComponentLink1URL (none) -> (none); ComponentLink2Description (none) -> (none); ComponentLink2URL (none) -> (none); CreateDate (none) -> 02/14/20 00:00:00; Database Table Name (none) -> ICs And Semiconductors; Device (none) -> 93C46B-I/SN; Footprint Library (none) -> ICs And Semiconductors SMD; Footprint Path (none) -> PcbLib\ICs And Semiconductors SMD.PcbLib; Footprint Ref (none) -> SOIC127P600X175-8N; HelpURL (none) -> \\cern.ch\dfs\Applications\Altium\Datasheets\93C46B-ISN.pdf; LatestRevisionDate (none) -> 02/14/20 00:00:00; Library Name (none) -> Logic; Library Path (none) -> SchLib\Logic.SchLib; Library Ref (none) -> 93C46B-SN; License (none) -> CC-BY-SA 4.0; Mounted (none) -> Yes; PackageDescription (none) -> SOIC, 1.27mm Pitch; 8 Pin - Body 4x5mm, IPC Medium Density; Part Description (none) -> 1Kbit, 5V, MICROWIRE® Serial EEPROM with 16-Bit Organization; Part Number (none) -> 93C46B-I_SN; Pin Count (none) -> 8; PressFit (none) -> No; SCEM (none) -> (none); SMD (none) -> Yes; Sense (none) -> No; Sense Comment (none) -> (none); Socket (none) -> No; Status (none) -> (none); Status Comment (none) -> (none)

Commit message: correcting some footprint issues
Parts:
- Y1: value OSC_25MHZ_RAKON_IVT3205CR -> 9132S-Y25.000N33DT1J
- Y6: value XTAL_25MHZ_TXC_8Y-25.000MAAJ-T -> ABM8W-25.0000MHZ-8-D1X-T3; footprint Footprint:XTAL_TXC_8Y -> Footprint:XTAL_ABM8W-25.0000MHZ-8-D1X-T3; Part Number XTAL_25MHZ_TXC_8Y-25.000MAAJ-T -> ABM8W-25.0000MHZ-8-D1X-T3
Changed lines of the file:
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@@
 			)
 		)
-		(property "Value" "XTAL_25MHZ_TXC_8Y-25.000MAAJ-T"
+		(property "Value" "ABM8W-25.0000MHZ-8-D1X-T3"
 			(at 177.8 147.955 0)
 			(effects
@@
 			)
 		)
-		(property "Footprint" "Footprint:XTAL_TXC_8Y"
+		(property "Footprint" "Footprint:XTAL_ABM8W-25.0000MHZ-8-D1X-T3"
 			(at 177.8 149.86 0)
 			(effects
@@
 			)
 		)
-		(property "Part Number" "XTAL_25MHZ_TXC_8Y-25.000MAAJ-T"
+		(property "Part Number" "ABM8W-25.0000MHZ-8-D1X-T3"
 			(at 177.8 153.67 0)
 			(effects
@@
 			)
 		)
-		(property "Value" "OSC_25MHZ_RAKON_IVT3205CR"
+		(property "Value" "9132S-Y25.000N33DT1J"
 			(at 105.41 37.846 0)
 			(effects
