File: Obsidian/FPGA_MISC.kicad_sch (KiCad schematic)
At the start: 21 parts, among them Q3 BSS138LT1G, SW1 SW_DIP_x01, U1 XC7A35T-CSG325, U27 S25FL128SAGMFI001, U9 REF3012

Commit message: revison v1.1.0 ready to review
Parts:
- removed R161: R0402_10K_1%_0.0625W_100PPM, Resistors SMD:RESC1005X40N, symbol Resistors SMD:R0402_10K_1%_0.0625W_100PPM
- added R161: R0402_4K7_1%_0.0625W_100PPM, Resistors SMD:RESC1005X40N, symbol Resistors SMD:R0402_4K7_1%_0.0625W_100PPM
Connections:
- net +3V3: now also R161.2
- net at LD5.2 (A): now also R161.1

Commit message: ready to manufacture
Connections:
- net FPGA_DONE: now reaches Q3.1 (G), U1.F12 (DONE_0)
Changed lines of the file:
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@@
+	)
+	(junction
+		(at 207.01 93.98)
+		(diameter 0)
+		(color 0 0 0 0)
 	)
 	(junction
@@
 	(wire
 		(pts
-			(xy 175.26 99.06) (xy 195.58 99.06)
+			(xy 175.26 99.06) (xy 212.09 99.06)
 		)
 		(stroke
@@
 		(pts
 			(xy 175.26 99.06) (xy 175.26 91.44)
+		)
+		(stroke
+			(width 0)
+			(type default)
+		)
+	)
+	(wire
+		(pts
+			(xy 207.01 93.98) (xy 212.09 93.98)
 		)
 		(stroke
@@
 		)
 	)
+	(global_label "FPGA_DONE"
+		(shape output)
+		(at 212.09 93.98 0)
+		(fields_autoplaced yes)
+		(effects
+			(font
+				(size 1.27 1.27)
+			)
+			(justify left)
+		)
+		(property "Intersheetrefs" "${INTERSHEET_REFS}"
+			(at 225.84 93.98 0)
+			(effects
+				(font
+					(size 1.27 1.27)
+				)
+				(justify left)
+				(hide yes)
+			)
+		)
+	)
 	(global_label "JTAG_TDO"
 		(shape output)
@@
 	(global_label "RST"
 		(shape input)
-		(at 195.58 99.06 0)
+		(at 212.09 99.06 0)
 		(fields_autoplaced yes)
 		(effects
@@
 		)
 		(property "Intersheetrefs" "${INTERSHEET_REFS}"
-			(at 202.0123 99.06 0)
+			(at 218.5223 99.06 0)
 			(effects
 				(font
