File: Obsidian/Ethernet.kicad_sch (KiCad schematic)
At the start: 42 parts, among them J3 BELFUSE_0826-1G1T-43-F, U7 RTL8211F-CG, Y4 XTAL_25MHZ_EPSON_TSX-3225_25.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

Commit message: Update schematic for out of stock components
Parts:
- R10, R11, R12, R13, R14, R15, R16, R17, R18: LCSC C25900 -> C2906869
- R4, R5, R6, R7, R8, R9: LCSC C25092 -> C114765
Changed lines of the file:
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@@
 			)
 		)
-		(property "Datasheet" "${KIPRJMOD}/datasheet/C25900.pdf"
+		(property "Datasheet" "${KIPRJMOD}/datasheet/C2906869.pdf"
 			(at 153.543 168.91 0)
 			(effects
@@
 			)
 		)
-		(property "LCSC" "C25900"
+		(property "LCSC" "C2906869"
 			(at 144.78 168.91 90)
 			(effects
@@
 			)
 		)
-		(property "Datasheet" "${KIPRJMOD}/datasheet/C25900.pdf"
+		(property "Datasheet" "${KIPRJMOD}/datasheet/C2906869.pdf"
 			(at 115.443 167.64 0)
 			(effects
@@
 			)
 		)
-		(property "LCSC" "C25900"
+		(property "LCSC" "C2906869"
 			(at 106.68 167.64 90)
 			(effects
@@
 			)
 		)
-		(property "Datasheet" "${KIPRJMOD}/datasheet/C25092.pdf"
+		(property "Datasheet" "${KIPRJMOD}/datasheet/C114765.pdf"
 			(at 55.88 120.523 0)
 			(effects
@@
 			)
 		)
-		(property "LCSC" "C25092"
+		(property "LCSC" "C114765"
 			(at 55.88 111.76 0)
 			(effects
@@
 			)
 		)
-		(property "Datasheet" "${KIPRJMOD}/datasheet/C25092.pdf"
+		(property "Datasheet" "${KIPRJMOD}/datasheet/C114765.pdf"
 			(at 55.88 111.633 0)
 			(effects
@@
 			)
 		)
-		(property "LCSC" "C25092"
+		(property "LCSC" "C114765"
 			(at 55.88 102.87 0)
 			(effects
@@
 			)
 		)
-		(property "Datasheet" "${KIPRJMOD}/datasheet/C25900.pdf"
+		(property "Datasheet" "${KIPRJMOD}/datasheet/C2906869.pdf"
 			(at 145.923 168.91 0)
 			(effects
@@
 			)
 		)
-		(property "LCSC" "C25900"
+		(property "LCSC" "C2906869"
 			(at 137.16 168.91 90)
 			(effects
@@
 			)
 		)
-		(property "Datasheet" "${KIPRJMOD}/datasheet/C25092.pdf"
+		(property "Datasheet" "${KIPRJMOD}/datasheet/C114765.pdf"
 			(at 55.88 117.983 0)
 			(effects
@@
 			)
 		)
-		(property "LCSC" "C25092"
+		(property "LCSC" "C114765"
 			(at 55.88 109.22 0)
 			(effects
@@
 			)
 		)
-		(property "Datasheet" "${KIPRJMOD}/datasheet/C25900.pdf"
+		(property "Datasheet" "${KIPRJMOD}/datasheet/C2906869.pdf"
 			(at 153.543 152.4 0)
 			(effects
@@
 			)
 		)
-		(property "LCSC" "C25900"
+		(property "LCSC" "C2906869"
 			(at 144.78 152.4 90)
 			(effects
@@
 			)
 		)
-		(property "Datasheet" "${KIPRJMOD}/datasheet/C25900.pdf"
+		(property "Datasheet" "${KIPRJMOD}/datasheet/C2906869.pdf"
 			(at 123.063 167.64 0)
 			(effects
@@
 			)
 		)
-		(property "LCSC" "C25900"
+		(property "LCSC" "C2906869"
 			(at 114.3 167.64 90)
 			(effects
@@
 			)
 		)
-		(property "Datasheet" "${KIPRJMOD}/datasheet/C25092.pdf"
+		(property "Datasheet" "${KIPRJMOD}/datasheet/C114765.pdf"
 			(at 55.88 106.553 0)
 			(effects
@@
 			)
 		)
-		(property "LCSC" "C25092"
+		(property "LCSC" "C114765"
 			(at 55.88 97.79 0)
 			(effects
@@
 			)
 		)
-		(property "Datasheet" "${KIPRJMOD}/datasheet/C25092.pdf"
+		(property "Datasheet" "${KIPRJMOD}/datasheet/C114765.pdf"
 			(at 55.88 114.173 0)
 			(effects
@@
 			)
 		)
-		(property "LCSC" "C25092"
+		(property "LCSC" "C114765"
 			(at 55.88 105.41 0)
 			(effects
@@
 			)
 		)
-		(property "Datasheet" "${KIPRJMOD}/datasheet/C25900.pdf"
+		(property "Datasheet" "${KIPRJMOD}/datasheet/C2906869.pdf"
 			(at 123.063 152.4 0)
 			(effects
@@
 			)
 		)
-		(property "LCSC" "C25900"
+		(property "LCSC" "C2906869"
 			(at 114.3 152.4 90)
 			(effects
@@
 			)
 		)
-		(property "Datasheet" "${KIPRJMOD}/datasheet/C25900.pdf"
+		(property "Datasheet" "${KIPRJMOD}/datasheet/C2906869.pdf"
 			(at 95.123 167.64 0)
 			(effects
@@
 			)
 		)
-		(property "LCSC" "C25900"
+		(property "LCSC" "C2906869"
 			(at 86.36 167.64 90)
 			(effects
@@
 			)
 		)
-		(property "Datasheet" "${KIPRJMOD}/datasheet/C25900.pdf"
+		(property "Datasheet" "${KIPRJMOD}/datasheet/C2906869.pdf"
 			(at 69.723 167.64 0)
 			(effects
@@
 			)
 		)
-		(property "LCSC" "C25900"
+		(property "LCSC" "C2906869"
 			(at 60.96 167.64 90)
 			(effects
@@
 			)
 		)
-		(property "Datasheet" "${KIPRJMOD}/datasheet/C25900.pdf"
+		(property "Datasheet" "${KIPRJMOD}/datasheet/C2906869.pdf"
 			(at 63.373 167.64 0)
 			(effects
@@
 			)
 		)
-		(property "LCSC" "C25900"
+		(property "LCSC" "C2906869"
 			(at 54.61 167.64 90)
 			(effects
@@
 			)
 		)
-		(property "Datasheet" "${KIPRJMOD}/datasheet/C25092.pdf"
+		(property "Datasheet" "${KIPRJMOD}/datasheet/C114765.pdf"
 			(at 55.88 109.093 0)
 			(effects
@@
 			)
 		)
-		(property "LCSC" "C25092"
+		(property "LCSC" "C114765"
 			(at 55.88 100.33 0)
 			(effects
